File: PiTFT32.brd (EAGLE design)
At the start: 85 x 116 mm, 64 parts, among them IC1 TP4056, IC2 TSC2046, Q1 A03400, Q3 BSS138, Q4 BSS138, X1 RASPI_BOARD_B+_F

Commit message: Update
Parts:
- removed BATT+, BATT+1, BATT-, BATT-1: (no value), wirepad:3,81/1,4
- removed C3, C4: 22UF, rcl:C1812K@1
- removed D24: (no value), Wurth_Elektronik_Optoelectronics_rev15c:3528
- removed IC1: TP4056, TP4056:SOP-8
- removed JP1: (no value), pinhead:1X04/90
- removed LED1: RED, led:CHIPLED_0805
- removed LED2, LED3: GREEN, led:CHIPLED_0805
- removed PAD1, PAD2: (no value), wirepad:SMD2,54-5,08
- removed PAD5, PAD6: (no value), wirepad:SMD1,27-2,54
- removed Q1: A03400, transistor-npn:SOT23-BEC
- removed Q3, Q4: BSS138, SparkFun:SOT23-3
- removed R10, R11, R8, R9: 10K, SparkFun:0603-RES
- removed R12, R13: 1k, SparkFun-Resistors:0603
- removed R14, R15: 2K, rcl:R1206
- removed R16, R17: 1K, rcl:R0603
- removed R2: 10R, adafruit:R0603
- removed R20, R4: 1K, rcl:R1206
- removed R3: 100K, adafruit:R0603
- removed R32, R33, R6, R7: 1K, SmartPrj:R0603-ROUND
- removed R34, R35: 10k, SmartPrj:R0603-ROUND
- removed R5: 100, rcl:R1206
- removed TP11: TPB2,54, testpad:B2,54
- removed U$1: FS312F-G, buckboost:SOT23-6
- removed U$2: TFT-DISPLAY-3.2-OB, tft32:TFT-DISPLAY-3.2-OB
- removed U$3: FS8205, buckboost:SOT23-6
- removed U$4: MT3608, buckboost:SOT23-6
- removed U$6: XKBENTERPRISESS-12D11G5R, XKB Enterprise SS-12D11G5R:XKBENTERPRISESS-12D11G5R
- added C7, C8: 10uF, SparkFun:EIA3216
- added CON1, CON25: Phoenix Pluggable 3.81mm 4 way, openbuilds-eagle-library:3.81MM-4WAY-PLUGGABLE-SCREW
- added D12: 5.1V1SMB5918BT3G9, diode:SMB
- added D7: SS34, semicon-smd-ipc:SOD87
- added IC4: (no value), linear:TO263-5
- added IC5: 1117-33, v-reg:SOT223
- added J2, J3: (no value), SparkFun-Connectors:2X5-SHROUDED
- added LOGO1: OSHW-LOGOM, SparkFun-Aesthetics:OSHW-LOGO-M
- added PAD3: (no value), wirepad:SMD2,54-5,08
- added Q2: A03400, transistor-npn:SOT23-BEC
- added R18: 10R, adafruit:R0603
- added R19: 100K, adafruit:R0603
- added R21, R22, R23, R24: 150R, SmartPrj:R0603-ROUND
- added R25, R26: 10k, SmartPrj:R0603-ROUND
- added TP1, TP5, TP6: TPB1,27, testpad:B1,27
- added U$5: TFT-DISPLAY-3.2-OB, tft32:TFT-DISPLAY-3.2-OB
- added X2: (no value), con-wago-500:W237-102
- C1: value 0.1UF -> (none); device rcl:C1206@1 -> resistor:E3,5-8
- C2: value 22UF -> (none); device rcl:C1812K@1 -> resistor:E3,5-8
- D1: value SS34 -> (none); device dp_devices:DO-214AC -> SparkFun-LED:LED_5MM
- J1: value (none) -> RJ45; device SparkFun-Connectors:USB-B-MICRO-SMD -> SparkFun-Connectors:RJ45-8
- L1: value 22UH -> 33uH; device rc-master-smd:CD75 -> inductors:DR127
- R1: value 7.5K -> 1k; device rcl:R1206 -> SparkFun-Resistors:AXIAL-0.3-KIT
- TP10, TP2, TP3, TP4, TP7, TP8, TP9: value TPB2,54 -> TPB1,27; device testpad:B2,54 -> testpad:B1,27
- X1: value RASPI_BOARD_B+_F -> RASPI_BOARD_B+_E0; device raspberrypi_bastelstube_v13:RASPI_BOARD_B+_FULL -> raspberrypi_bastelstube_v13:RASPI_BOARD_B+_EDGES_0DRILL
- moved C1 377.5 mm to (81.0, 46.6), turned to 90 degrees
- moved R1 345.5 mm to (70.7, 80.5), flipped to the bottom, turned to 0 degrees
- moved D1 338.5 mm to (69.1, 86.1), flipped to the bottom, turned to 270 degrees
- moved L1 328.7 mm to (75.3, 35.6), turned to 180 degrees
- moved C2 321.3 mm to (72.5, 46.6), turned to 90 degrees
- moved J1 302.4 mm to (76.0, 82.5)
- moved X1 265.5 mm to (118.0, 3.50), turned to 90 degrees
- moved TP3 185.2 mm to (60.1, 37.1), flipped to the top
- moved TP4 183.9 mm to (58.4, 34.3), flipped to the top
- moved TP2 182.6 mm to (60.2, 35.2), flipped to the top, turned to 0 degrees
- moved TP7 180.0 mm to (58.5, 36.1), flipped to the top
- moved TP8 179.3 mm to (58.5, 38.0), flipped to the top, turned to 0 degrees
- moved TP10 177.2 mm to (58.5, 40.0), flipped to the top, turned to 0 degrees
- moved TP9 176.8 mm to (60.3, 33.3), flipped to the top, turned to 0 degrees
- moved R62 174.8 mm to (49.4, 32.6), turned to 270 degrees
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Connections:
- net 3V3 renamed N$1
- removed net 5V0: X1.2
- removed net 5V_BOOST: C3.2, D1.1, LED3.A, PAD1.1, R1.2
- removed net 5V_HEADER: JP1.1
- removed net BATT+: BATT+.1, BATT+1.1, IC1.5, R5.2, U$6.CENTER
- removed net BATT-: BATT-.1, BATT-1.1, C1.1, U$1.6, U$3.1
- removed net CHG: IC1.7, R17.2
- removed net FEEDBACK5V: R1.1, R4.2, U$4.3
- removed net LEDCHR: LED1.C, R17.1
- removed net LEDSBY: LED2.C, R16.1
- removed net N$1 (its old number): Q1.B, R2.1, R3.1
- removed net N$11: D24.3, R12.2
- removed net N$15: U$2.P$1
- removed net N$18: R7.2, U$2.P$12
- removed net N$20: R32.2, U$2.P$13
- removed net N$21: D24.4, R13.2
- removed net N$22: R33.2, U$2.P$14
- removed net N$7: LED3.C, R20.1
- removed net N$9: R6.2, U$2.P$11
- removed net OC: U$1.3, U$3.4
- removed net OD: U$1.1, U$3.6
- removed net PROG: IC1.2, R15.1
- removed net RXEXT: JP1.3, Q3.3, R9.2
- removed net STANDBY: IC1.6, R16.2
- removed net SWITCH5V: D1.2, L1.1, U$4.1
- removed net TXEXT: JP1.4, Q4.3, R11.2
- removed net V-IN-BOOST: C2.2, L1.2, U$4.4, U$4.5, U$6.RIGHT
- removed net VCC-PROT: C1.2, R5.1, U$1.5
- removed net VUSB: C4.1, IC1.4, IC1.8, J1.VBUS, LED1.A, LED2.A, PAD6.1
- new net BL: CON1.1, J1.4
- new net BL1: R21.2, U$5.P$11, U$5.P$29
- new net BL2: R22.2, U$5.P$12, U$5.P$30
- new net BL3: R23.2, U$5.P$13, U$5.P$31
- new net BL4: R24.2, U$5.P$14, U$5.P$32
- new net BLWH: CON25.1, J1.5
- new net BR: CON25.3, J1.8
- new net BRWH: CON25.2, J1.7
- new net GR: CON25.4, J1.6
- new net GRWH: CON1.4, J1.3
- new net HI-V-IN: C1.+, IC4.1, X2.2
- new net N$3: Q2.B, R18.1, R19.1
- new net N$8: D7.1, IC4.2, L1.1
- new net OR: CON1.2, J1.2
- new net ORWH: CON1.3, J1.1
- net 16_RXD2: no longer Q3.2, R12.1, R8.2
- net 17_TXD2: no longer Q4.2, R10.2, R13.1
- net 3.3V: now also C8.A, IC5.4, R25.1, R26.1, U$5.P$27, U$5.P$9; no longer D24.1, D24.2, Q3.1, Q4.1, R10.1, R34.1, R35.1, R8.1, U$2.P$9
- net 5V_L2: now also C2.+, C7.A, D1.A, D12.C, IC4.4, IC5.3, J2.2, J3.2, L1.2, TP6.TP, U$5.P$10, U$5.P$28, X1.2; no longer R11.1, R9.1, U$2.P$10
- net BACKLIGHT: now also J2.8, J3.8, R18.2, TP9.TP; no longer R2.2, TP4.TP
- net BACKLIGHTGND: now also Q2.C, R21.1, R22.1, R23.1, R24.1; no longer Q1.C, R32.1, R33.1, R6.1, R7.1
- net GND: now also C1.-, C2.-, C7.C, C8.C, D12.A, D7.2, IC4.3, IC4.5, IC4.6, IC5.1, J2.1, J3.1, Q2.E, R1.P$1, R19.2, TP1.TP, U$5.P$1, U$5.P$19, U$5.P$26, U$5.P$8, X2.1; no longer C2.1, C3.1, C4.2, IC1.1, IC1.3, J1.D+, J1.GND, J1.ID, J1.SHIELD1, J1.SHIELD2, J1.SHIELD3, JP1.2, PAD2.1, PAD5.1, Q1.E, R14.1, R15.2, R20.2, R3.2, R4.1, U$2.P$8, U$3.3, U$4.2
- net N$2: now also D1.K, R1.P$2; no longer R14.2, U$1.2
- net SPI_CE0: now also J2.6, J3.6, U$5.P$23, U$5.P$5; no longer U$2.P$5
- net SPI_CE1: now also J2.9, J3.9, TP5.TP; no longer TP3.TP
- net SPI_MISO: now also J2.4, J3.4, TP7.TP, U$5.P$25, U$5.P$7; no longer TP2.TP, U$2.P$7
- net SPI_MOSI: now also J2.3, J3.3, TP2.TP, U$5.P$24, U$5.P$6; no longer TP7.TP, U$2.P$6
- net SPI_SCK: now also J2.5, J3.5, TP3.TP, U$5.P$21, U$5.P$3; no longer TP10.TP, U$2.P$3
- net TFT_DC: now also J2.7, J3.7, R25.2, TP4.TP, U$5.P$22, U$5.P$4; no longer R34.2, TP9.TP, U$2.P$4
- net TFT_RST: now also PAD3.1, R26.2, U$5.P$2, U$5.P$20; no longer R35.2, TP11.TP, U$2.P$2, X1.13
- net TOUCHIRQ: now also J2.10, J3.10, TP10.TP
- net X+: now also U$5.P$17, U$5.P$35; no longer U$2.P$17
- net X-: now also U$5.P$15, U$5.P$33; no longer U$2.P$15
- net Y+: now also U$5.P$16, U$5.P$34; no longer U$2.P$16
- net Y-: now also U$5.P$18, U$5.P$36; no longer U$2.P$18
Routing:
- net 5V_L2: track 0.00 -> 228.4 mm, vias 0 -> 6
- net TFT_DC: track 0.00 -> 175.1 mm, vias 0 -> 6
- net SPI_MOSI: track 0.00 -> 164.2 mm, vias 0 -> 6
- net SPI_SCK: track 0.00 -> 160.7 mm, vias 0 -> 7
- net SPI_MISO: track 0.00 -> 160.4 mm, vias 0 -> 7
- net SPI_CE0: track 0.00 -> 154.8 mm, vias 0 -> 7
- net BACKLIGHT: track 0.00 -> 149.2 mm, vias 0 -> 4
- net TOUCHIRQ: track 0.00 -> 120.9 mm, vias 0 -> 4
- net SPI_CE1: track 0.00 -> 120.1 mm, vias 0 -> 5
- net 3.3V: track 0.00 -> 66.0 mm, vias 0 -> 2
- net GND: track 0.00 -> 65.4 mm, vias 0 -> 84
- net TFT_RST: track 0.00 -> 55.0 mm, vias 0 -> 2
- net HI-V-IN: track 0.00 -> 43.6 mm, vias 0 -> 1
- net X-: track 0.00 -> 24.3 mm, vias 0 -> 3
- net Y+: track 0.00 -> 23.0 mm, vias 0 -> 3
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- added copper zone on layer 1, net 5V_L2
- added copper zone on layer 1, net GND
- added copper zone on layer 16, net GND
- added copper zone on layer 1, net HI-V-IN
- added copper zone on layer 1, net N$8
Other:
- board size 85 x 116 mm -> 96.5 x 99 mm
- board text added: "+"
- board text added: "-"
- board text added: "BLUE"
- board text added: "BLWH"
- board text added: "BRN"
- board text added: "BRNWH"
- board text added: "DESIGNED BY PETER VAN DER WALT (2021)"
- board text added: "GPLv3"
- board text added: "GRN"
- board text added: "GRWH"
- board text added: "OR"
- board text added: "ORWH"
- board text added: "RASPBERRY PI GPIO HEADER"
- board text added: "RASPBERRY PI LCD ILI9341 WITH TOUCH TP2046"
- board text removed: "10K=130mA 5K=250mA 4K=300mA 3K=400mA 2K=580mA 1K66=690mA 1K5=780mA 1K33=900mA 1K2=1000mA"
- board text removed: "CHRG RATE"
