File: PiTFT32.sch (EAGLE design)
At the start: 64 parts, among them IC1 TP4056, IC2 TSC2046, Q1 A03400, Q3 BSS138, Q4 BSS138, X1 RASPI_BOARD_B+_F

Commit message: Update
Parts:
- removed BATT+, BATT+1, BATT-, BATT-1: (no value), wirepad:3,81/1,4
- removed C3, C4: 22UF, rcl:C-EUC1812K
- removed D24: (no value), Wurth_Elektronik_Optoelectronics_rev15c:WL-SBTW-150141RB73100-R&B
- removed IC1: TP4056, TP4056:TP4056
- removed JP1: (no value), pinhead:PINHD-1X4/90
- removed LED1: RED, led:LEDCHIPLED_0805
- removed LED2, LED3: GREEN, led:LEDCHIPLED_0805
- removed PAD1, PAD2: (no value), wirepad:SMD5
- removed PAD5, PAD6: (no value), wirepad:SMD2
- removed Q1: A03400, transistor-npn:BC849SMD
- removed Q3, Q4: BSS138, SparkFun:MOSFET-NCHANNELSMD
- removed R10, R11, R8, R9: 10K, SparkFun:RESISTOR0603-RES
- removed R12, R13: 1k, SparkFun-Resistors:1KOHM-0603-1/10W-1%
- removed R14, R15: 2K, rcl:R-EU_R1206
- removed R16, R17: 1K, rcl:R-EU_R0603
- removed R2: 10R, adafruit:R-US_R0603
- removed R20, R4: 1K, rcl:R-EU_R1206
- removed R3: 100K, adafruit:R-US_R0603
- removed R32, R33, R7: 1K, SmartPrj:R-EU_R0603
- removed R34, R35: 10k, SmartPrj:R-EU_R0603
- removed R5: 100, rcl:R-EU_R1206
- removed R6: 1K, SmartPrj:R-EU_0603-RND
- removed TP11: TPB2,54, testpad:TPB2,54
- removed U$1: FS312F-G, buckboost:FS312F-G
- removed U$2: TFT-DISPLAY-3.2-OB, tft32:TFT-DISPLAY-3.2-OB
- removed U$3: FS8205, buckboost:FS8205
- removed U$4: MT3608, buckboost:MT3608
- removed U$6: XKBENTERPRISESS-12D11G5R, XKB Enterprise SS-12D11G5R:XKBENTERPRISESS-12D11G5R
- added C7, C8: 10uF, SparkFun:CAP_POL1206
- added CON1, CON25: Phoenix Pluggable 3.81mm 4 way, openbuilds-eagle-library:CONNECTOR-M4
- added D12: 5.1V1SMB5918BT3G9, diode:ZENER-DIODESMB
- added D7: SS34, semicon-smd-ipc:D-SOD-87
- added IC4: (no value), linear:LM2596S
- added IC5: 1117-33, v-reg:LD117AS33TR
- added J2, J3: (no value), SparkFun-Connectors:CONN_05X2SHD
- added LOGO1: OSHW-LOGOM, SparkFun-Aesthetics:OSHW-LOGOM
- added PAD3: (no value), wirepad:SMD5
- added Q2: A03400, transistor-npn:BC849SMD
- added R18: 10R, adafruit:R-US_R0603
- added R19: 100K, adafruit:R-US_R0603
- added R21: 150R, SmartPrj:R-EU_0603-RND
- added R22, R23, R24: 150R, SmartPrj:R-EU_R0603
- added R25, R26: 10k, SmartPrj:R-EU_R0603
- added TP1, TP5, TP6: TPB1,27, testpad:TPB1,27
- added U$5: TFT-DISPLAY-3.2-OB, tft32:TFT-DISPLAY-3.2-OB
- added X2: (no value), con-wago-500:W237-102
- C1: value 0.1UF -> (none); device rcl:C-EUC1206 -> resistor:CPOL-EUE3.5-8
- C2: value 22UF -> (none); device rcl:C-EUC1812K -> resistor:CPOL-EUE3.5-8
- D1: value SS34 -> (none); device dp_devices:DIODE-DO-214AC -> SparkFun-LED:LED5MM
- J1: value (none) -> RJ45; device SparkFun-Connectors:USB_MICRO-B_FEMALE-SMT -> SparkFun-Connectors:RJ45-8
- L1: value 22UH -> 33uH; device rc-master-smd:L_CD75 -> inductors:DR127
- R1: value 7.5K -> 1k; device rcl:R-EU_R1206 -> SparkFun-Resistors:1KOHM-HORIZ_KIT-1/4W-5%
- TP10, TP2, TP3, TP4, TP7, TP8, TP9: value TPB2,54 -> TPB1,27; device testpad:TPB2,54 -> testpad:TPB1,27
- X1: value RASPI_BOARD_B+_F -> RASPI_BOARD_B+_E0; device raspberrypi_bastelstube_v13:RASPI_BOARD_B+_F -> raspberrypi_bastelstube_v13:RASPI_BOARD_B+_E0
Connections:
- removed net 5V_BOOST: C3.2, D1.C, LED3.A, PAD1.P, R1.2
- removed net 5V_HEADER: JP1.1
- removed net BATT+: BATT+.P, BATT+1.P, IC1.BAT, R5.2, U$6.CENTER
- removed net BATT-: BATT-.P, BATT-1.P, C1.1, U$1.GND, U$3.S1
- removed net CHG: IC1.CHRG, R17.2
- removed net FEEDBACK5V: R1.1, R4.2, U$4.FB
- removed net LEDCHR: LED1.C, R17.1
- removed net LEDSBY: LED2.C, R16.1
- removed net N$11: D24.C1, R12.2
- removed net N$15: U$2.1_GND
- removed net N$18: R7.2, U$2.12_LEDK
- removed net N$20: R32.2, U$2.13_LEDK
- removed net N$21: D24.C2, R13.2
- removed net N$22: R33.2, U$2.14_LEDK
- removed net N$7: LED3.C, R20.1
- removed net N$9: R6.2, U$2.11_LEDK
- removed net OC: U$1.OC, U$3.G2
- removed net OD: U$1.OD, U$3.G1
- removed net PROG: IC1.PROG, R15.1
- removed net RXEXT: JP1.3, Q3.D, R9.2
- removed net STANDBY: IC1.STDBY, R16.2
- removed net SWITCH5V: D1.A, L1.1, U$4.SW
- removed net TXEXT: JP1.4, Q4.D, R11.2
- removed net V-IN-BOOST: C2.2, L1.2, U$4.EN, U$4.VIN, U$6.RIGHT
- removed net VCC-PROT: C1.2, R5.1, U$1.VCC
- removed net VUSB: C4.1, IC1.CE, IC1.VCC, J1.VBUS, LED1.A, LED2.A, PAD6.P
- new net BL: CON1.1, J1.4
- new net BL1: R21.2, U$5.11_LEDK
- new net BL2: R22.2, U$5.12_LEDK
- new net BL3: R23.2, U$5.13_LEDK
- new net BL4: R24.2, U$5.14_LEDK
- new net BLWH: CON25.1, J1.5
- new net BR: CON25.3, J1.8
- new net BRWH: CON25.2, J1.7
- new net GR: CON25.4, J1.6
- new net GRWH: CON1.4, J1.3
- new net HI-V-IN: C1.+, IC4.IN, X2-2.KL
- new net N$3: Q2.B, R18.1, R19.1
- new net N$8: D7.C, IC4.OUT, L1.1
- new net OR: CON1.2, J1.2
- new net ORWH: CON1.3, J1.1
- net 16_RXD2: no longer Q3.S, R12.1, R8.2
- net 17_TXD2: no longer Q4.S, R10.2, R13.1
- net 3.3V: now also C8.+, IC5.OUT, R25.1, R26.1, U$5.9_VCC; no longer D24.A1, D24.A2, Q3.G, Q4.G, R10.1, R34.1, R35.1, R8.1, U$2.9_VCC
- net 5V_L2: now also C2.+, C7.+, D1.A, D12.C, IC4.FB, IC5.IN, J2.2, J3.2, L1.2, TP6.TP, U$5.10_LEDA, X1.5V0; no longer R11.1, R9.1, U$2.10_LEDA
- net BACKLIGHT: now also J2.8, J3.8, R18.2, TP9.TP; no longer R2.2, TP4.TP
- net BACKLIGHTGND: now also Q2.C, R21.1, R22.1, R23.1, R24.1; no longer Q1.C, R32.1, R33.1, R6.1, R7.1
- net GND: now also C1.-, C2.-, C7.-, C8.-, D12.A, D7.A, IC4.EN, IC4.GND, IC4.GND@1, IC5.ADJ, J2.1, J3.1, Q2.E, R1.1, R19.2, TP1.TP, U$5.1_GND, U$5.8_GND, X2-1.KL; no longer C2.1, C3.1, C4.2, IC1.GND, IC1.TEMP, J1.D+, J1.GND, J1.ID, J1.SHIELD, JP1.2, PAD2.P, PAD5.P, Q1.E, R14.1, R15.2, R20.2, R3.2, R4.1, U$2.8_GND, U$3.S2, U$4.GND
- net N$1: now also X1.3V3; no longer Q1.B, R2.1, R3.1
- net N$2: now also D1.C, R1.2; no longer R14.2, U$1.CS
- net SPI_CE0: now also J2.6, J3.6, U$5.5_CS; no longer U$2.5_CS
- net SPI_CE1: now also J2.9, J3.9, TP5.TP; no longer TP3.TP
- net SPI_MISO: now also J2.4, J3.4, TP7.TP, U$5.7_SDO; no longer TP2.TP, U$2.7_SDO
- net SPI_MOSI: now also J2.3, J3.3, TP2.TP, U$5.6_SDA; no longer TP7.TP, U$2.6_SDA
- net SPI_SCK: now also J2.5, J3.5, TP3.TP, U$5.3_SCL; no longer TP10.TP, U$2.3_SCL
- net TFT_DC: now also J2.7, J3.7, R25.2, TP4.TP, U$5.4_RS/A0; no longer R34.2, TP9.TP, U$2.4_RS/A0
- net TFT_RST: now also PAD3.P, R26.2, U$5.2_RESET; no longer R35.2, TP11.TP, U$2.2_RESET, X1.GPIO27
- net TOUCHIRQ: now also J2.10, J3.10, TP10.TP
- net X+: now also U$5.17_X+; no longer U$2.17_X+
- net X-: now also U$5.15_X-; no longer U$2.15_X-
- net Y+: now also U$5.16_Y-; no longer U$2.16_Y-
- net Y-: now also U$5.18_Y+; no longer U$2.18_Y+
Other:
- note removed: "+"
- note removed: "-"
- note removed: "From https://circuits4you.com/2018/12/31/esp32-hardware-serial2-example/ #define RXD2 16 #define TXD2 17"
- note removed: "RX TO EXTERNAL DEVICE (COMES FROM TX ON GRBL)"
- note removed: "Serial Port 5v"
- note removed: "TX FROM EXTERNAL DEVICE (GOES TO RX ON GRBL)"
